File: RF_HUNTER.kicad_sch (KiCad schematic)
At the start: 0 parts

Commit message: Added all the important files to PCB manufacturing
Parts:
- added 2.4GHz1, 5GHz1: Conn_Coaxial, Library:CON-SMA-EDGE, symbol Connector:Conn_Coaxial
- added C1, C2, C4, C7: 100pF, Capacitor_SMD:C_0402_1005Metric_Pad0.74x0.62mm_HandSolder, symbol Device:C
- added C5: 2pF, Capacitor_SMD:C_0402_1005Metric_Pad0.74x0.62mm_HandSolder, symbol Device:C
- added C6: 100nF, Capacitor_SMD:C_0402_1005Metric_Pad0.74x0.62mm_HandSolder, symbol Device:C
- added R1: 68Ω, Resistor_SMD:R_0402_1005Metric_Pad0.72x0.64mm_HandSolder, symbol Device:R
- added R2: 10kΩ, Resistor_SMD:R_0402_1005Metric_Pad0.72x0.64mm_HandSolder, symbol Device:R
- added R3: 20kΩ, Resistor_SMD:R_0402_1005Metric_Pad0.72x0.64mm_HandSolder, symbol Device:R
- added U2: (no value), Library:GRF1201, symbol RF_Hunter_Needed:GRF1201
- added U3: HMC849A, footprints:CP_16_40_ADI-M, symbol RF_Switch:HMC849A
- added U4: ESP32-DevKitC, Connector_PinSocket_2.54mm:PinSocket_1x04_P2.54mm_Vertical, symbol PCM_Espressif:ESP32-DevKitC
- added unknown1: ?, Resistor_SMD:R_0402_1005Metric_Pad0.72x0.64mm_HandSolder, symbol Device:C
Connections:
- new net: U3.1 (VDD), unknown1.2
- new net: C1.1, U3.12 (RF2)
- new net: U3.2 (VCTL), U4.11 (ADC2_CH7/GPIO27)
- new net: C5.1, R1.2, U3.3 (RFC)
- new net: C2.1, U3.9 (RF1)
- new net: 5GHz1.1 (In), C1.2
- new net: 2.4GHz1.1 (In), C2.2
- new net: C4.2, C6.1, C7.1, U2.6 (VCC), U4.19 (5V), unknown1.1
- new net: R2.1, R3.2, U2.4 (DC_Out)
- new net: R2.2, U4.5 (VDET_1/GPIO34/ADC1_CH6)
- new net: C5.2, U2.3 (RF_In)
- new net GND: 2.4GHz1.2 (Ext), 5GHz1.2 (Ext), C4.1, C6.2, C7.2, R1.1, R3.1, U2.1 (NC/GND), U2.2 (NC/GND), U2.5 (NC/GND), U3.10 (GND), U3.11 (GND), U3.13 (GND), U3.14 (GND), U3.15 (GND), U3.16 (GND), U3.17 (GND), U3.4 (GND), U3.5 (EN), U3.6 (GND), U3.7 (GND), U3.8 (GND), U4.14 (GND), U4.32 (GND), U4.38 (GND)
